File: nixie.kicad_pcb (KiCad board)
At the start: 4 copper layers, 102.6 x 65.2 mm, 28 parts, among them IC1 SN74141, IC2 SN74141, IC3 SN74141, IC4 SN74141, IC5 MIC5219-5.0YM5-TR, IC6 DS3231M+TRL, J1 1984989

Commit message: Add files via upload
Parts:
- N1, N2, N3, N4: value IN-14 -> Val**
- U$1: renamed from THE pi
Changed lines of the file:
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@@
     (property "ki_description" "LDO Voltage Regulators 500mA Peak 1% Low Noise LDO")
     (attr smd)
-    (fp_text reference "IC5" (at 0 0 180) (layer "F.SilkS") hide
+    (fp_text reference "IC5" (at 0 0 180) (layer "F.SilkS")
         (effects (font (size 1.27 1.27) (thickness 0.254)))
     )
@@
         (effects (font (size 1.27 1.27) (thickness 0.254)))
     )
-    (fp_text user "${REFERENCE}" (at 0.782 2.728 180) (layer "F.SilkS")
+    (fp_text user "${REFERENCE}" (at -0.5 -2.8 180) (layer "F.Fab")
         (effects (font (size 1.27 1.27) (thickness 0.254)))
     )
@@
     (property "Sheetfile" "nixie.kicad_sch")
     (property "Sheetname" "")
-    (fp_text reference "N4" (at 0 -1.016 90) (layer "B.SilkS")
-        (effects (font (size 1.1684 1.1684) (thickness 0.1016)) (justify right bottom mirror))
+    (fp_text reference "N4" (at -0.94 0.9 270) (layer "F.SilkS")
+        (effects (font (size 1.1684 1.1684) (thickness 0.1016)) (justify right bottom))
     )
-    (fp_text value "IN-14" (at 0 0) (layer "B.Fab") hide
+    (fp_text value "Val**" (at 0 0) (layer "B.Fab") hide
         (effects (font (size 1.27 1.27) (thickness 0.15)) (justify mirror))
     )
-    (fp_arc (start 7.6201 0) (mid -0.07935 7.54065) (end -7.62 -0.1588)
-      (stroke (width 0.254) (type solid)) (layer "B.SilkS"))
+    (fp_arc (start 7.6201 0) (mid -0.07935 7.540649) (end -7.62 -0.1588)
+      (stroke (width 0.254) (type solid)) (layer "F.SilkS"))
     (fp_circle (center 0 0) (end 8.8744 0)
-      (stroke (width 0.254) (type solid)) (fill none) (layer "B.SilkS"))
+      (stroke (width 0.254) (type solid)) (fill none) (layer "F.SilkS"))
     (pad "0" thru_hole circle (at 5.0942 -3.5163 180) (size 1.348 1.348) (drill 0.84) (layers "*.Cu" "*.Mask")
       (net 48 "/N40") (pinfunction "0") (pintype "bidirectional") (solder_mask_margin 0.1016))
@@
     (property "Sheetfile" "nixie.kicad_sch")
     (property "Sheetname" "")
-    (fp_text reference "THE pi" (at 0.47 9.23 -270) (layer "B.SilkS")
+    (fp_text reference "U$1" (at 0.47 9.23 -270) (layer "B.SilkS")
         (effects (font (size 1.27 1.27) (thickness 0.15)) (justify mirror))
     )
@@
     (property "Sheetfile" "nixie.kicad_sch")
     (property "Sheetname" "")
-    (fp_text reference "N3" (at 0 -1.016 90) (layer "B.SilkS")
-        (effects (font (size 1.1684 1.1684) (thickness 0.1016)) (justify right bottom mirror))
+    (fp_text reference "N3" (at 54.7413 1.1 270) (layer "F.SilkS")
+        (effects (font (size 1.1684 1.1684) (thickness 0.1016)) (justify right bottom))
     )
-    (fp_text value "IN-14" (at 0 0) (layer "B.Fab") hide
+    (fp_text value "Val**" (at 0 0) (layer "B.Fab") hide
         (effects (font (size 1.27 1.27) (thickness 0.15)) (justify mirror))
     )
-    (fp_arc (start 7.6201 0) (mid -0.07935 7.54065) (end -7.62 -0.1588)
-      (stroke (width 0.254) (type solid)) (layer "B.SilkS"))
+    (fp_arc (start 7.6201 0) (mid -0.07935 7.540649) (end -7.62 -0.1588)
+      (stroke (width 0.254) (type solid)) (layer "F.SilkS"))
     (fp_circle (center 0 0) (end 8.8744 0)
-      (stroke (width 0.254) (type solid)) (fill none) (layer "B.SilkS"))
+      (stroke (width 0.254) (type solid)) (fill none) (layer "F.SilkS"))
     (pad "0" thru_hole circle (at 5.0942 -3.5163 180) (size 1.348 1.348) (drill 0.84) (layers "*.Cu" "*.Mask")
       (net 34 "/N30") (pinfunction "0") (pintype "bidirectional") (solder_mask_margin 0.1016))
@@
     (property "Sheetfile" "nixie.kicad_sch")
     (property "Sheetname" "")
-    (fp_text reference "N1" (at -0.0142 -1.016 90) (layer "B.SilkS")
-        (effects (font (size 1.1684 1.1684) (thickness 0.1016)) (justify right bottom mirror))
+    (fp_text reference "N1" (at -55.3658 0.7 270) (layer "F.SilkS")
+        (effects (font (size 1.1684 1.1684) (thickness 0.1016)) (justify right bottom))
     )
-    (fp_text value "IN-14" (at 0 0) (layer "B.Fab") hide
+    (fp_text value "Val**" (at 0 0) (layer "B.Fab") hide
         (effects (font (size 1.27 1.27) (thickness 0.15)) (justify mirror))
     )
-    (fp_arc (start 7.6201 0) (mid -0.07935 7.54065) (end -7.62 -0.1588)
-      (stroke (width 0.254) (type solid)) (layer "B.SilkS"))
+    (fp_arc (start 7.6201 0) (mid -0.07935 7.540649) (end -7.62 -0.1588)
+      (stroke (width 0.254) (type solid)) (layer "F.SilkS"))
     (fp_circle (center 0 0) (end 8.8744 0)
-      (stroke (width 0.254) (type solid)) (fill none) (layer "B.SilkS"))
+      (stroke (width 0.254) (type solid)) (fill none) (layer "F.SilkS"))
     (pad "0" thru_hole circle (at 5.0942 -3.5163 180) (size 1.348 1.348) (drill 0.84) (layers "*.Cu" "*.Mask")
       (net 6 "/N10") (pinfunction "0") (pintype "bidirectional") (solder_mask_margin 0.1016))
@@
     (property "Sheetfile" "nixie.kicad_sch")
     (property "Sheetname" "")
-    (fp_text reference "N2" (at 0 -1.27 90) (layer "B.SilkS")
-        (effects (font (size 1.1684 1.1684) (thickness 0.1016)) (justify right bottom mirror))
+    (fp_text reference "N2" (at -0.904 0.7 270) (layer "F.SilkS")
+        (effects (font (size 1.1684 1.1684) (thickness 0.1016)) (justify right bottom))
     )
-    (fp_text value "IN-14" (at 0 0) (layer "B.Fab") hide
+    (fp_text value "Val**" (at 0 0) (layer "B.Fab") hide
         (effects (font (size 1.27 1.27) (thickness 0.15)) (justify mirror))
     )
-    (fp_arc (start 7.6201 0) (mid -0.07935 7.54065) (end -7.62 -0.1588)
-      (stroke (width 0.254) (type solid)) (layer "B.SilkS"))
+    (fp_arc (start 7.6201 0) (mid -0.07935 7.540649) (end -7.62 -0.1588)
+      (stroke (width 0.254) (type solid)) (layer "F.SilkS"))
     (fp_circle (center 0 0) (end 8.8744 0)
-      (stroke (width 0.254) (type solid)) (fill none) (layer "B.SilkS"))
+      (stroke (width 0.254) (type solid)) (fill none) (layer "F.SilkS"))
     (pad "0" thru_hole circle (at 5.0942 -3.5163 180) (size 1.348 1.348) (drill 0.84) (layers "*.Cu" "*.Mask")
       (net 20 "/N20") (pinfunction "0") (pintype "bidirectional") (solder_mask_margin 0.1016))

Commit message: Adding WIP files
Parts:
- added IC5: MCP23017-E_SO, L7805CV:SOIC127P1030X265-28N, F.Cu at (66.4, 111.1)
- added IC9: L7805CV, L7805CV:TO255P460X1020X2008-3P, F.Cu at (76.2, 105.2)
- N1, N2, N3, N4: value Val** -> IN-14
Connections:
- U$1 pad GP10: /A3 -> unconnected-(U$1-PadGP10)
- U$1 pad GP11: /D3 -> unconnected-(U$1-PadGP11)
- U$1 pad GP12: /B3 -> unconnected-(U$1-PadGP12)
- U$1 pad GP13: /C3 -> unconnected-(U$1-PadGP13)
- U$1 pad GP14: /A4 -> unconnected-(U$1-PadGP14)
- U$1 pad GP15: /D4 -> unconnected-(U$1-PadGP15)
- U$1 pad GP16: /C4 -> unconnected-(U$1-PadGP16)
- U$1 pad GP17: /B4 -> unconnected-(U$1-PadGP17)
- U$1 pad GP2: /A1 -> /SDA1
- U$1 pad GP3: /D1 -> /SCL1
- U$1 pad GP4: /B1 -> unconnected-(U$1-PadGP4)
- U$1 pad GP5: /C1 -> unconnected-(U$1-PadGP5)
- U$1 pad GP6: /A2 -> unconnected-(U$1-PadGP6)
- U$1 pad GP7: /D2 -> unconnected-(U$1-PadGP7)
- U$1 pad GP8: /B2 -> unconnected-(U$1-PadGP8)
- U$1 pad GP9: /C2 -> unconnected-(U$1-PadGP9)

Commit message: revert
Parts:
- removed the IC5 at (66.4, 111.1)
- removed IC9: L7805CV, L7805CV:TO255P460X1020X2008-3P
- N1, N2, N3, N4: value IN-14 -> Val**
Connections:
- U$1 pad GP10: unconnected-(U$1-PadGP10) -> /A3
- U$1 pad GP11: unconnected-(U$1-PadGP11) -> /D3
- U$1 pad GP12: unconnected-(U$1-PadGP12) -> /B3
- U$1 pad GP13: unconnected-(U$1-PadGP13) -> /C3
- U$1 pad GP14: unconnected-(U$1-PadGP14) -> /A4
- U$1 pad GP15: unconnected-(U$1-PadGP15) -> /D4
- U$1 pad GP16: unconnected-(U$1-PadGP16) -> /C4
- U$1 pad GP17: unconnected-(U$1-PadGP17) -> /B4
- U$1 pad GP2: /SDA1 -> /A1
- U$1 pad GP3: /SCL1 -> /D1
- U$1 pad GP4: unconnected-(U$1-PadGP4) -> /B1
- U$1 pad GP5: unconnected-(U$1-PadGP5) -> /C1
- U$1 pad GP6: unconnected-(U$1-PadGP6) -> /A2
- U$1 pad GP7: unconnected-(U$1-PadGP7) -> /D2
- U$1 pad GP8: unconnected-(U$1-PadGP8) -> /B2
- U$1 pad GP9: unconnected-(U$1-PadGP9) -> /C2
